File: Hardware/Power.kicad_sch (KiCad schematic)
At the start: 49 parts, among them J2 JST_2mm_LiPo, Q2 SIL2308, Q4 BSS138, Q5 BSS138, U10 MCP73833_MSOP, U11 AP2112K-3.3, U12 STLQ015-3.3, U14 74LVC1G175, U4 MAX17048, U5 AP2112K-3.3, U6 74LVC1G14, U8 74LVC1G17

Commit message: Update 3D models
Parts:
- U10: footprint SparkFun-Semiconductor-Standard:MSOP-10 -> SparkFun-Semiconductor-Standard:MSOP-10_3x3mm_P0.5mm
Changed lines of the file:
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@@
 			)
 		)
-		(property "Footprint" "SparkFun-Semiconductor-Standard:MSOP-10"
+		(property "Footprint" "SparkFun-Semiconductor-Standard:MSOP-10_3x3mm_P0.5mm"
 			(at 72.39 73.66 0)
 			(effects
