File: Hardware/Power.kicad_sch (KiCad schematic)
At the start: 51 parts, among them J2 JST_2mm_LiPo, Q2 SIL2308, Q4 BSS138, Q5 BSS138, U10 MCP73833_MSOP, U11 AP2112K-3.3, U12 STLQ015-3.3, U14 SN74LVC1G175DCK, U4 MAX17048, U6 SN74LVC1G14DCK, U7 AP7361C-3.3V, U8 SN74LVC1G17DCK

Commit message: Add JST PROD_IDs. Update AP7361C regulator
Parts:
- U7: Ityp (none) -> 1.0A
Changed lines of the file:
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@@
 			)
 		)
-		(property "Description" "600mA low dropout linear adjustable regulator, with enable pin, 2.2-6.0V input, 0.8-5.0V output, UDFN-8"
+		(property "Description" "1A low dropout linear regulator, with enable pin, 2.2-6.0V input, 3.3V output, UDFN-8"
 			(at 112.014 205.232 0)
 			(effects
@@
 			(at 113.03 218.44 0)
 			(effects
+				(font
+					(size 1.27 1.27)
+				)
+				(hide yes)
+			)
+		)
+		(property "Ityp" "1.0A"
+			(at 113.03 218.44 0)
+			(effects
