File: Hardware/SparkFun_RTK_Facet_mosaic.kicad_sch (KiCad schematic)
At the start: 28 parts, among them J3 Qwiic_RA, J5 Conn_01x12_FPC_0.5mm, J6 Conn_01x12_FPC_0.5mm, J7 Conn_01x12_FPC_0.5mm, U1 ESP32-WROVER-E-N16R8

Commit message: V1.1 Panelized
Parts:
- removed U7: ~, SparkFun-Aesthetic:Ordering_Instructions, symbol SparkFun-Aesthetic:Ordering_Instructions
Connections:
- net ESP18/MEventB: now reaches U1.30 (IO18)
Changed lines of the file:
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@@
 	(title_block
 		(title "RTK Facet L-Band mosaic")
-		(date "2024-01-23")
+		(date "2024-05-02")
 		(rev "v11")
 		(comment 1 "Designed by: N.S. & P.C.")
@@
 	(wire
 		(pts
+			(xy 95.25 148.59) (xy 96.52 148.59)
+		)
+		(stroke
+			(width 0)
+			(type default)
+		)
+	)
+	(wire
+		(pts
 			(xy 34.29 62.23) (xy 34.29 64.77)
 		)
@@
 				)
 				(justify right)
+				(hide yes)
+			)
+		)
+	)
+	(global_label "ESP18{slash}MEventB"
+		(shape input)
+		(at 96.52 148.59 0)
+		(fields_autoplaced yes)
+		(effects
+			(font
+				(size 1.27 1.27)
+			)
+			(justify left)
+		)
+		(property "Intersheetrefs" "${INTERSHEET_REFS}"
+			(at 113.2331 148.59 0)
+			(effects
+				(font
+					(size 1.27 1.27)
+				)
+				(justify left)
 				(hide yes)
 			)
@@
 					(unit 1)
 				)
-			)
-		)
-	)
-	(symbol
-		(lib_id "SparkFun-Aesthetic:Ordering_Instructions")
-		(at 254 185.42 0)
-		(unit 1)
-		(exclude_from_sim no)
-		(in_bom yes)
-		(on_board yes)
-		(dnp no)
-		(fields_autoplaced yes)
-		(property "Reference" "U7"
-			(at 254 182.88 0)
-			(effects
-				(font
-					(size 1.27 1.27)
-				)
-				(hide yes)
-			)
-		)
-		(property "Value" "~"
-			(at 254 185.42 0)
-			(effects
-				(font
-					(size 1.27 1.27)
-				)
-				(hide yes)
-			)
-		)
-		(property "Footprint" "SparkFun-Aesthetic:Ordering_Instructions"
-			(at 254 185.42 0)
-			(effects
-				(font
-					(size 1.27 1.27)
-				)
-				(hide yes)
-			)
-		)
-		(property "Datasheet" ""
-			(at 254 185.42 0)
-			(effects
-				(font
-					(size 1.27 1.27)
-				)
-				(hide yes)
-			)
-		)
-		(property "Description" ""
-			(at 254 185.42 0)
-			(effects
-				(font
-					(size 1.27 1.27)
-				)
-				(hide yes)
-			)
-		)
-		(instances
-			(project "SparkFun_RTK_Facet_mosaic"
-				(path "/e3dd3ae4-244d-4cba-9cca-5d2abf83f29a"
-					(reference "U7")
-					(unit 1)
-				)
