File: Hardware/GNSS.kicad_sch (KiCad schematic)
At the start: 27 parts, among them J1 U.FL, Q3 BSS138, U13 74HC4052D, U2 mosaic-X5

Commit message: v1.2 routed
Parts:
- D1: value TVS_0402 -> PESD0402
Other:
- title: (none) -> GNSS
Changed lines of the file:
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@@
 	(generator_version "8.0")
 	(paper "USLetter")
+	(title_block
+		(title "GNSS")
+	)
 	(junction
 		(at 64.77 182.88)
@@
 			)
 		)
-		(property "Value" "TVS_0402"
+		(property "Value" "PESD0402"
 			(at 219.71 48.26 90)
 			(effects
@@
 			)
 		)
-		(property "Datasheet" "~"
+		(property "Datasheet" "https://docs.sparkfun.com/SparkFun_RTK_mosaic-X5/assets/component_documentation/Mosaic%20Hardware%20Manual_v1.8.0.pdf"
 			(at 68.58 138.43 0)
 			(effects
