File: Hardware/SparkFun_RTK_Facet_mosaic.kicad_pcb (KiCad board)
At the start: 4 copper layers, 59.5 x 43 mm, 172 parts, among them J1 U.FL, J2 JST_2mm_LiPo, J3 Qwiic_RA, J5 Conn_01x12_FPC_0.5mm, J6 Conn_01x12_FPC_0.5mm, J7 Conn_01x12_FPC_0.5mm, Q1 MBT3904DW1, Q2 SIL2308, Q3 BSS138, Q4 BSS138, Q5 BSS138, U1 ESP32-WROVER-E-N16R8, U10 MCP73833_MSOP, U11 AP2112K-3.3, U12 STLQ015-3.3, U13 74HC4052D, U14 74LVC1G175, U2 mosaic-X5, U3 CH340C, U4 MAX17048, U5 AP2112K-3.3, U6 74LVC1G14, U8 74LVC1G17, U9 USB251xB, Y1 24MHz

Commit message: v1.2 routed
Parts:
- removed J6, J7: Conn_01x12_FPC_0.5mm, SparkFun-Connector:FPC_0.5mm-12
- removed R40: 10k, SparkFun-Resistor:R_0402_1005Metric
- removed kibuzzard-65776CDC: G***, kibuzzard-65776CDC
- removed kibuzzard-65776CEB: G***, kibuzzard-65776CEB
- removed kibuzzard-65776CEF: G***, kibuzzard-65776CEF
- removed kibuzzard-65776CF4: G***, kibuzzard-65776CF4
- added D6: BAS16J, SparkFun-Semiconductor-Standard:SOD-323, B.Cu at (138.9, 147.7)
- added J4: Conn_01x12, SparkFun-Connector:JST_SMD_1.0mm-12_RA, F.Cu at (138.1, 117.2)
- added R42: 100k, SparkFun-Resistor:R_0402_1005Metric, B.Cu at (140.7, 147.4)
- added R43: 100k, SparkFun-Resistor:R_0402_1005Metric, B.Cu at (120.9, 141.9)
- D1: value TVS_0402 -> PESD0402
- D2: value TVS_ESD_4_HS -> DF5A5.6LFU
- D3, D4: value 3A -> BAT60A
- FID1, FID2, FID3, FID4: value Fiducial_0.5 -> Fiducial_0.5mm
- J5: value Conn_01x12_FPC_0.5mm -> Conn_01x14; footprint SparkFun-Connector:FPC_0.5mm-12 -> SparkFun-Connector:JST_SMD_1.0mm-14_RA
- R10: value 10k -> 100k
- U10: footprint SparkFun-Semiconductor-Standard:MSOP-10 -> SparkFun-Semiconductor-Standard:MSOP-10_3x3mm_P0.5mm
- U14: value 74LVC1G175 -> SN74LVC1G175DCK
- U6: value 74LVC1G14 -> SN74LVC1G14DCK
- U8: value 74LVC1G17 -> SN74LVC1G17DCK
- moved R10 30.3 mm to (109.5, 138.4), turned to 180 degrees
- moved C26 18.4 mm to (143.1, 117.2), turned to 0 degrees
- moved U13 8.00 mm to (136.3, 116.7), turned to 90 degrees
- moved kibuzzard-65A7F686 7.22 mm to (123.6, 116.8)
- moved C17 6.19 mm to (146.7, 148.5)
- moved TP19 4.58 mm to (121.9, 116.8)
- moved J1 4.21 mm to (127.9, 115.2)
- moved D2 4.00 mm to (144.2, 114.7), turned to 180 degrees
- moved D4 3.86 mm to (144.7, 135.8), turned to -90 degrees
- moved J5 3.69 mm to (116.6, 117.2)
- moved D1 3.22 mm to (128.4, 118.1), turned to 180 degrees
- moved R28 2.90 mm to (144.4, 120.0)
- moved R37 2.90 mm to (143.4, 120.0)
- moved R38 2.90 mm to (142.4, 120.0)
- moved D3 2.79 mm to (141.2, 134.6), turned to 180 degrees
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Connections:
- C17 pad 1: VIN -> VUSB
- D3 pad A: VBATT -> VUSB
- D4 pad A: VUSB -> VBATT
- J5 pad 10: GND -> USB_DM
- J5 pad 11: GND -> MRX2
- J5 pad 12: GND -> MTX2
- J5 pad 3: VUSB -> VRAW
- J5 pad 4: VUSB -> ExternalDATA_RXI
- J5 pad 5: unconnected-(J5-Pin_5-Pad5) -> ExternalDATA_TXO
- J5 pad 6: VRAW -> ESP22/SCL
- J5 pad 7: VRAW -> ESP21/SDA
- J5 pad 8: VRAW -> 3.3V_P
- J5 pad 9: VRAW -> USB_DP
- R10 pad 2: ESP34/CHG_LED -> ESP19/CHG_STAT2
- U1 pad 31: ESP19/CHG_LED2 -> ESP19/CHG_STAT2
- U1 pad 6: ESP34/CHG_LED -> ESP34/CHG_STAT1
- U10 pad 1: VIN -> VUSB
- U10 pad 2: VIN -> VUSB
- U10 pad 3: ESP34/CHG_LED -> CHG_LED
- U10 pad 4: ESP19/CHG_LED2 -> ESP19/CHG_STAT2
Routing:
- net CHG_LED: track 0.00 -> 59.6 mm, vias 0 -> 3
- net ESP34/CHG_LED: track 51.4 -> 0.00 mm, vias 5 -> 0
- net ESP19/CHG_LED2: track 50.4 -> 0.00 mm, vias 4 -> 0
- net ESP19/CHG_STAT2: track 0.00 -> 48.0 mm, vias 0 -> 4
- net ESP34/CHG_STAT1: track 0.00 -> 38.0 mm, vias 0 -> 4
- net VIN: track 102.3 -> 67.5 mm
- net ExternalDATA_RXI: track 33.1 -> 57.9 mm, vias 2 -> 3
- net MRX3: track 53.4 -> 29.7 mm
- net MPPS_3V3: track 70.9 -> 52.4 mm, vias 3 -> 1
- net VUSB: track 172.8 -> 155.5 mm, vias 7 -> 8
- net MEventA: track 50.3 -> 34.8 mm
- net 3.3V: track 122.2 -> 109.9 mm, vias 15 -> 12
- net ESP39/ADC39: track 28.9 -> 40.6 mm, vias 3 -> 4
- net ESP26/DAC2: track 28.7 -> 39.9 mm, vias 1 -> 3
- net USB_DM: track 8.21 -> 19.1 mm
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Other:
- board text added: "v1.2"
- board text removed: "v11"

Commit message: v1.2 Panelized
Parts:
- moved Ref** 53.2 mm to (114.9, 149.2)
- moved kibuzzard-65A7F7BA 0.76 mm to (145.0, 139.8)
- moved kibuzzard-65A7F7EA 0.76 mm to (145.0, 144.7)
- moved kibuzzard-65776D0F 0.18 mm to (154.9, 132.5)
Routing:
- net ExternalDATA_RXI: track 57.9 -> 56.9 mm
- net MTX2: track 62.2 -> 63.1 mm
- net ExternalDATA_TXO: track 43.9 -> 43.1 mm
- net ESP~{RST}: track 44.3 -> 44.8 mm
- net GND: vias 141 -> 147

Commit message: Add SD_DET and 1A regulator
Parts:
- removed U5: AP2112K-3.3, SparkFun-Semiconductor-Standard:SOT23-5
- added TP24: 1.0mm, SparkFun-Connector:TestPoint-1.0mm, B.Cu at (157.5, 144.8)
- added TP25: 1.0mm, SparkFun-Connector:TestPoint-1.0mm, B.Cu at (157.5, 142.2)
- added U7: AP7361C-3.3V, SparkFun-Semiconductor-Standard:UDFN-8, B.Cu at (131.6, 141.6)
- added kibuzzard-670CFFCD: G***, kibuzzard-670CFFCD, B.Cu at (155.6, 142.2)
- added kibuzzard-670CFFE9: G***, kibuzzard-670CFFE9, B.Cu at (155.6, 144.8)
- moved D1 0.38 mm to (128.4, 118.5)
- moved J1 0.25 mm to (127.9, 115.4)
- turned C21 to 180 degrees
- turned C7 to 180 degrees
Connections:
- J4 pad 4: 3.3V_P -> ESP15/SD_~{DET}
- U1 pad 23: unconnected-(U1-IOA15-Pad23) -> ESP15/SD_~{DET}
Routing:
- net ESP15/SD_~{DET}: track 0.00 -> 48.2 mm, vias 0 -> 2
- net VRAW: track 116.9 -> 120.9 mm
- net MTX2: track 63.1 -> 65.6 mm, vias 2 -> 3
- net MRX2: track 63.3 -> 65.9 mm, vias 2 -> 3
- net ESP39/ADC39: track 40.6 -> 42.2 mm
- net GND: track 78.0 -> 76.6 mm, vias 147 -> 150
- net ESP27/PeripheralPower: track 19.5 -> 20.7 mm, vias 2 -> 3
- net VBATT: track 62.1 -> 62.7 mm
- net 3.3V_P: track 203.3 -> 203.8 mm, vias 13 -> 12

Commit message: Add JST PROD_IDs. Update AP7361C regulator
Parts:
- J1: value U.FL -> Val**
- TR1: value RFCMF1220100M4T -> Val**
Changed lines of the file:
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@@
 			)
 		)
-		(property "Value" "U.FL"
+		(property "Value" "Val**"
 			(at 0 2.2 -90)
 			(layer "F.Fab")
@@
 		)
 		(group ""
-			(members "046ac3b2-c7c1-4495-ac29-6f14273c2e89" "0534dcf1-80e1-4bc2-8b87-2fc6bee82f0a"
-				"3a015d72-893f-472e-ad5b-303ad81cab8e" "52762fdf-fbf1-4295-bec5-c94ff92565b9"
-				"7b875d5c-6394-4308-941b-bd4256fff1ac" "7fdba089-056f-4d4f-80fd-cde671677b33"
-				"e800777f-1737-4c3c-a0d5-b54375d107dd" "fa202280-8645-4ed5-bc5d-d9f6a95b1ecf"
-				"fa4f4f6f-24f8-4f81-b106-8174e8ce817b"
+			(members "1c1c69f0-a11a-4ed0-9bb9-20cfb8dd9c4b" "69a664be-355c-4ff1-a2a7-5ee911d3f928"
+				"6fe202a4-6600-4086-8b36-5b50e62aa656" "855ea946-bf8a-4082-8fa6-776b6e00084c"
+				"a2403eab-749f-4780-bd55-e0b8c4f565bf" "a78e5320-b4a0-4f94-ae1a-5f58f8e11184"
+				"d23e13e0-c04e-4346-b440-bae8a2338acd" "f44d0595-69d2-4c02-b520-ec7551c28d21"
+				"fabd32e8-0fa9-4c25-81fb-008ccfc72000"
 			)
 		)
@@
 			)
 		)
-		(property "PROD_ID" "..."
+		(property "PROD_ID" "CONN-23694"
 			(at 0 0 180)
 			(unlocked yes)
@@
 		)
 		(group ""
-			(members "1f03aca1-324a-4176-9aa3-c1d05a003413" "4383f481-9407-42b1-b719-969d453b625a"
-				"4bb244d7-150d-4c99-b835-78e2b836adf7" "574196f5-fddb-4b9c-abee-ba9206057977"
-				"9758e3cc-5c41-4d7f-8005-331bb71eb2e9" "d59f28ab-011b-4306-a7e2-9d313ce5abd6"
-				"ddb0373c-31f5-49f0-a0b8-feb03fce3308" "e93ef243-f9c5-4ec8-940a-3ac015994a34"
+			(members "08808e3a-685f-41d5-b5bd-8842899ee517" "0c57d787-51c8-4924-8563-82c0cf4b779f"
+				"7e0a6bfd-9d22-4537-9f1c-aa11f26607b1" "a2ccbe91-6273-4387-8d77-2cf84dbe3eca"
+				"a633a044-dff8-4186-af61-0659b78f727a" "ed8ba82b-4685-4219-8297-183d97363689"
+				"f7c18589-c1e8-4298-9311-9cec0219f7c3" "fc85e40a-88d2-4201-94a3-c3f3edd80eb2"
 			)
 		)
@@
 			)
 		)
-		(property "PROD_ID" "..."
+		(property "PROD_ID" "CONN-23695"
 			(at 0 0 180)
 			(unlocked yes)
@@
 		(sheetfile "SparkFun_RTK_Facet_mosaic.kicad_sch")
 		(attr exclude_from_bom)
-		(fp_text user " https://creativecommons.org/licenses/by-sa/4.0/"
-			(at 0 1.27 0)
+		(fp_text user "Released under the Creative Commons Attribution Share-Alike 4.0 License"
+			(at 0 -1.27 0)
 			(layer "F.Fab")
 			(effects
@@
 			)
 		)
-		(fp_text user "Released under the Creative Commons Attribution Share-Alike 4.0 License"
-			(at 0 -1.27 0)
+		(fp_text user " https://creativecommons.org/licenses/by-sa/4.0/"
+			(at 0 1.27 0)
 			(layer "F.Fab")
 			(effects
@@
 		)
 		(group ""
-			(members "6bc3bd93-1dbc-4649-8fd3-72ef521e7634")
+			(members "0542e151-ec7f-4412-b39d-81aad925e009")
 		)
 	)
@@
 				(font
 					(size 0.001 0.001)
+					(thickness 0.15)
 				)
 				(justify mirror)
@@
 				(font
 					(size 0.001 0.001)
+					(thickness 0.15)
 				)
 				(justify mirror)
@@
 				(font
 					(size 0.001 0.001)
+					(thickness 0.15)
 				)
 				(justify mirror)
@@
 				(font
 					(size 0.001 0.001)
+					(thickness 0.15)
 				)
 				(justify mirror)
@@
 		)
 		(group ""
-			(members "32b442af-fc7e-42d6-a003-b7b0f567261d" "5b99e641-fc69-4efa-a761-0dd0ec6ef691"
-				"77168c1f-63a4-4082-9a69-718f25a0a859" "b2ac8608-f9b1-4d76-a144-044889d53859"
-				"c69a90f0-511f-4f1c-8557-6ce612862640" "d06bccae-97b6-497e-8943-a295a9c633e7"
-				"d4986ed5-ee5e-4951-8ed1-d665ce9b7791" "e013ffc6-fe58-4fed-94e9-1f980a96d3f2"
-				"e5690ea3-0dbd-4492-8371-95bad0462581"
+			(members "186acd0e-54ef-4605-9db7-dbed4d3b57d8" "2a6cc034-1f73-4d62-b23f-3f7c7cf8b5df"
+				"2f6555b1-7625-46bf-b1cc-01ffb19cad59" "374a5b25-9abb-47dd-936d-758b3b22524f"
+				"683af842-4ac2-4102-bc0e-0890575711ee" "6e86a110-ca64-4a3c-9166-471ea9637a54"
+				"854863ec-f414-44ac-9d05-1307068cd30d" "de3af444-32d9-46b2-8db3-9d64c94c26d6"
+				"ea0526fb-d5ec-400c-8e76-241822b272ea"
 			)
 		)
@@
 		(fp_arc
 			(start 1.9463 4.8768)
-			(mid 1.834732 5.146223)
+			(mid 1.834737 5.146237)
 			(end 1.5653 5.257777)
 			(stroke
@@
 		(fp_arc
 			(start 1.9463 4.8768)
-			(mid 1.834732 5.146223)
+			(mid 1.834737 5.146237)
 			(end 1.5653 5.257777)
 			(stroke
@@
 			)
 		)
-		(property "Value" "RFCMF1220100M4T"
+		(property "Value" "Val**"
 			(at 0 -1.2 0)
 			(layer "B.Fab")
@@
 			)
 		)
-		(property "Description" "600mA low dropout linear adjustable regulator, with enable pin, 2.2-6.0V input, 0.8-5.0V output, UDFN-8"
+		(property "Description" "1A low dropout linear regulator, with enable pin, 2.2-6.0V input, 3.3V output, UDFN-8"
 			(at 0 0 0)
 			(unlocked yes)
@@
 			)
 		)
+		(property "Ityp" "1.0A"
+			(at 0 0 90)
+			(unlocked yes)
+			(layer "B.Fab")
+			(hide yes)
+			(effects
+				(font
+					(size 1 1)
+					(thickness 0.15)
+				)
+				(justify mirror)
+			)
+		)
 		(property ki_fp_filters "SOT?23?5*")
 		(sheetname "Power")
@@
 			(thermal_bridge_angle 0)
 		)
+		(model "${SPARKFUN_KICAD_LIBRARY}/Footprints/SparkFun-3D-models/Semiconductor-Standard/DFN-8_3x3mm_P0.65mm.step"
+			(offset
+				(xyz 0 0 0.15)
+			)
+			(scale
+				(xyz 1 1 1)
+			)
+			(rotate
+				(xyz 90 0 180)
+			)
+		)
 	)
 	(footprint "SparkFun-Semiconductor-Standard:SOT23-5"
@@
 		(tags "SparkFun capacitor")
 		(property "Reference" "C21"
-			(at 0 1.16 360)
+			(at 0 1.16 0)
 			(layer "B.Fab")
 			(effects
@@
 		)
 		(property "Value" "1.0uF"
-			(at 0 -1.16 360)
+			(at 0 -1.16 0)
 			(layer "B.Fab")
 			(effects
